Commit message: 新增: 底盘偏航关节 base_yaw_joint, 工作空间扩展为桌面圆环区域
- 底座上加旋转塔台 yaw_link, 整条手臂可绕 Z 轴 ±3.14 rad 旋转
- 这样 A/B 两点不必都在手臂正前方的同一条弧线上, 可分布在桌面不同方位
- wrist_pitch 限位从 ±1.2 放宽到 ±1.5 rad, 增大可达范围余量
- arm_controller 关节列表与演示脚本同步更新

File: urdf/robomaster_ep_gazebo.urdf (robot description, URDF)
Before this commit: robot robomaster_ep_core, 7 links, 6 joints
Links:
- added link yaw_link, mass 0.3; collision cylinder length=0.08 radius=0.05; visual cylinder length=0.08 radius=0.05
Joints:
- added joint base_yaw_joint: type revolute, parent base_link, child yaw_link, origin xyz=0 0 0.14 rpy=0 0 0, axis 0 0 1, limit lower=-3.14 upper=3.14 effort=10 velocity=2.0
- joint arm_lift_joint: origin xyz=0.18 0 0.16 rpy=0 0 0 -> xyz=0.18 0 0.02 rpy=0 0 0; parent base_link -> yaw_link
- joint wrist_pitch_joint: limit lower=-1.2 upper=1.2 effort=10 velocity=1.0 -> lower=-1.5 upper=1.5 effort=10 velocity=1.0

Commit message: 修复验收联调三处问题 + 视觉升级: 官方 mesh 移植进 URDF
联调修复:
- pick_place 节点不再重复 declare use_sim_time (launch 已传入, 否则
  ParameterAlreadyDeclaredException 直接崩溃)
- ompl 管线 adapter 名改为 humble 正确名 AddTimeOptimalParameterization
  (AddTimeParameterization 不存在, 每次规划都报加载异常)

视觉升级 (官方 robomaster_ros mesh, 116 个 dae 已入库):
- 底盘: chassis/armor/battery/电池插销/控制器/盖板 + 4 个麦克纳姆轮
- 塔台: 云台球头/侧板/装甲板/底座环 + 水弹枪全套 + 扬声器
- 悬臂: 两片三角腹板连接塔台与抬臂轴, arm_base 底座块包住抬臂轴
- 上臂/前臂: arm_1/arm_2 mesh 经锚点求解 (抬臂轴/腕轴/腕托轴三点对齐)
- 夹爪: endpoint_bracket 腕托 + gripper_base 手掌 + 手指三段拉直排布
- 碰撞盒全部保留 (与官方底盘尺寸对齐后微缩 base 碰撞盒)
- 新增 tools/gen_mesh_visuals.py: DAE 包围盒 + 锚点变换求解工具

File: urdf/robomaster_ep_gazebo.urdf (robot description, URDF)
Before this commit: robot robomaster_ep_core, 8 links, 7 joints
Links:
- link base_link: geometry collision box size=0.34 0.22 0.10; visual mesh filename=package://robomaster_pick_place_sim/meshes/armor.dae scale=1 1 1
- link gripper_base_link: geometry collision box size=0.06 0.13 0.04; visual mesh filename=package://robomaster_pick_place_sim/meshes/endpoint_bracket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 scale=0.9685 0.9685 0.9685
- link left_finger_link: geometry collision box size=0.12 0.018 0.035; visual mesh filename=package://robomaster_pick_place_sim/meshes/gripper_left_1.d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 scale=1.26 1.26 1.26
- link right_finger_link: geometry collision box size=0.12 0.018 0.035; visual mesh filename=package://robomaster_pick_place_sim/meshes/right_gripper_1.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 scale=1.26 1.26 1.26
- link upper_arm_link: geometry collision box size=0.28 0.035 0.06; visual mesh filename=package://robomaster_pick_place_sim/meshes/arm_1.dae scale=2.1749 2.1749 2.1749
- link wrist_link: geometry collision box size=0.20 0.035 0.045; visual mesh filename=package://robomaster_pick_place_sim/meshes/arm_2.dae scale=1.5834 1.5834 1.5834
- link yaw_link: geometry collision cylinder length=0.08 radius=0.05; visual cylinder length=0.08 radius=0.05

Commit message: Replace root package with verified gripper-fixed model

File: urdf/robomaster_ep_gazebo.urdf (robot description, URDF)
Before this commit: robot robomaster_ep_core, 7 links, 6 joints
Links:
- added link yaw_link, mass 0.3; collision cylinder length=0.08 radius=0.05; visual mesh filename=package://robomaster_pick_place_sim/meshes/arm_base.dae scale=1 1 1
- link base_link: geometry collision box size=0.34 0.22 0.10; visual mesh filename=package://robomaster_pick_place_sim/meshes/armor.dae scale=1 1 1
- link gripper_base_link: geometry collision box size=0.06 0.13 0.04; visual mesh filename=package://robomaster_pick_place_sim/meshes/endpoint_bracket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 scale=1 1 1
- link left_finger_link: geometry collision box size=0.12 0.018 0.035; visual mesh filename=package://robomaster_pick_place_sim/meshes/gripper_left_1.d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 scale=1 1 1
- link right_finger_link: geometry collision box size=0.12 0.018 0.035; visual mesh filename=package://robomaster_pick_place_sim/meshes/right_gripper_1.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 scale=1 1 1
- link upper_arm_link: geometry collision box size=0.28 0.035 0.06; visual mesh filename=package://robomaster_pick_place_sim/meshes/arm_1.dae scale=1 1 1
- link wrist_link: geometry collision box size=0.20 0.035 0.045; visual mesh filename=package://robomaster_pick_place_sim/meshes/arm_2.dae scale=1 1 1
Joints:
- added joint base_yaw_joint: type revolute, parent base_link, child yaw_link, origin xyz=0 0.0010384 0.1152522 rpy=0 0 0, axis 0 0 1, limit lower=0 upper=0 effort=10 velocity=2.0
- joint arm_lift_joint: origin xyz=0.18 0 0.16 rpy=0 0 0 -> xyz=0.0103961 -0.0255713 0.030741 rpy=0 0 0; parent base_link -> yaw_link
- joint left_finger_joint: origin xyz=0.03 0.035 0 -> xyz=0.0163032 0.0212032 -0.0399201 rpy=0 0 0
- joint right_finger_joint: origin xyz=0.03 -0.035 0 -> xyz=0.0163034 -0.0209781 -0.0399201 rpy=0 0 0
- joint wrist_pitch_joint: limit lower=-1.2 upper=1.2 effort=10 velocity=1.0 -> lower=-1.5 upper=1.5 effort=10 velocity=1.0; origin xyz=0.28 0 0 -> xyz=0.0018704 0.0438659 0.1210238 rpy=0 0 0
- joint wrist_to_gripper: origin xyz=0.22 0 0 -> xyz=0.1058557 0.006752 -0.0561093 rpy=0 0 0
